File: kicad/arc_module/arc_module.kicad_pcb (KiCad board)
At the start: 2 copper layers, 100 x 100 mm, 80 parts, among them J1 CONN_01X07, J10 CONN_01X03, J11 CONN_01X03, J2 CONN_01X02, J3 CONN_01X03, J4 CONN_01X03, J6 CONN_01X03, J7 CONN_01X03, J8 CONN_01X03, J9 CONN_01X03, P1 pcie_1x_edge, P3 CONN_01X02, P4 CONN_01X01, P5 CONN_01X01, P6 CONN_01X01, Q1 BC847, Q2 NTR4502, U1 74HCT157, U2 74HCT157, U3 EP91H0, U4 PCA9500, U5 CS8416

Commit message: draft layout
Parts:
- added P7: CONN_01X01, Pin_Headers:Pin_Header_Straight_1x01_Pitch2.54mm, F.Cu at (127.3, 109.5)
- added P8: CONN_01X01, Pin_Headers:Pin_Header_Straight_1x01_Pitch2.54mm, F.Cu at (97.0, 125.2)
- added R36: 47k, Resistors_SMD:R_0805_HandSoldering, F.Cu at (98.8, 66.4)
- moved J3 100.2 mm to (90.7, 102.4)
- moved P4 100.0 mm to (165.6, 50.4), turned to 180 degrees
- moved P5 96.5 mm to (165.6, 84.6), turned to 180 degrees
- moved P3 96.4 mm to (165.6, 55.4), turned to 0 degrees
- moved J1 95.3 mm to (163.1, 50.4), turned to 0 degrees
- moved P6 92.4 mm to (165.6, 65.6), turned to 180 degrees
- moved D3 89.5 mm to (164.4, 70.7), turned to 180 degrees
- moved J7 88.7 mm to (90.7, 98.3)
- moved J8 88.6 mm to (90.7, 91.7)
- moved J6 87.8 mm to (103.4, 101.9)
- moved R35 86.2 mm to (162.1, 77.0), turned to 90 degrees
- moved R34 83.5 mm to (159.0, 84.0), turned to 90 degrees
- moved R33 80.2 mm to (159.3, 77.0), turned to 90 degrees
- moved L4 79.3 mm to (159.3, 71.3), turned to 90 degrees
- moved L3 75.8 mm to (157.3, 65.6), turned to 90 degrees
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Connections:
- L2 pad 2: +3.3VA -> +3V3
Routing:
- net GND: track 0.00 -> 101.8 mm, vias 0 -> 39
- net +3V3: track 0.00 -> 78.1 mm, vias 0 -> 12
- net VDDA: track 0.00 -> 54.4 mm, vias 0 -> 2
- net /CS8416/LR_clk: track 76.7 -> 30.8 mm
- net /Module Common/I2S0_mod: track 4.18 -> 48.0 mm
- net /CS8416/S_clk: track 66.8 -> 31.6 mm
- net /Module Common/SCL: track 0.00 -> 33.5 mm
- net +5V: track 0.00 -> 33.3 mm
- net /Module Common/SDA: track 0.00 -> 32.7 mm, vias 0 -> 1
- net /Module Common/IO0: track 0.00 -> 31.6 mm, vias 0 -> 3
- net /CS8416/M_clk: track 62.4 -> 31.9 mm
- net /SPD_Rx: track 0.00 -> 29.7 mm
- net /Module Common/Mclk_in: track 0.00 -> 25.8 mm
- net /Module Common/I2S3_in: track 0.00 -> 23.6 mm
- net /Module Common/Mclk_out: track 0.00 -> 23.0 mm, vias 0 -> 1
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- added copper zone on F.Cu, net +3V3
- added copper zone on B.Cu, net GND
Other:
- board size 100 x 100 mm -> 100 x 85 mm
- net class power added: clearance 0.2, trace_width 0.5, via_dia 0.6, via_drill 0.4
- board text added: "Need to copy cuts from other module for edge conenctor. (Could make a footprint that includes cuts??)"

Commit message: silkscreen & test points
Parts:
- added P10: CONN_01X02, Pin_Headers:Pin_Header_Straight_1x02_Pitch2.54mm, F.Cu at (165.6, 106.2)
- added P9: CONN_01X01, Pin_Headers:Pin_Header_Straight_1x01_Pitch2.54mm, F.Cu at (146.6, 77.7)
- moved R10 7.12 mm to (142.2, 109.5)
- moved J6 3.69 mm to (103.6, 105.5)
- moved R14 3.08 mm to (145.0, 117.9)
- moved R13 3.06 mm to (145.0, 121.2)
- moved J4 2.42 mm to (92.6, 58.3)
- moved J2 1.55 mm to (105.2, 114.8)
- moved R9 0.76 mm to (132.1, 55.6)
Routing:
- net /Module Common/I2S1_mod: track 22.6 -> 16.5 mm
- net /Tx_En: track 12.5 -> 16.5 mm
- net /CS8416/PDUR: track 10.2 -> 13.8 mm
- net Net-(R1-Pad2): track 0.00 -> 3.58 mm
- net /Module Common/I2S2_mod: track 9.16 -> 6.01 mm
- net /Module Common/I2S3_mod: track 9.08 -> 6.22 mm
- net /CS8416/RM/NV: track 5.43 -> 8.22 mm
- net VDDA: track 54.4 -> 57.2 mm
- net /Module Common/SCL: track 33.5 -> 31.9 mm
- net /Module Common/SDA: track 32.7 -> 31.1 mm
- net GND: track 101.8 -> 102.8 mm, vias 39 -> 38
Other:
- board text added: "13"
- board text added: "19"
- board text added: "3v3"
- board text added: "Err"
- board text added: "Gnd"
- board text added: "HDMI"
- board text added: "Modular Open-Source AV Receiver HDMI ARC Module [version 0] Andrew Bolin. 2017-04-23"
- board text added: "NV"
- board text added: "PDUR"
- board text added: "Power"
- board text added: "RMCF"
- board text added: "Rx"
- board text added: "SDA SCL"
- board text added: "SFSEL0"
- board text added: "SFSEL1"
- board text added: "SPDIF"
- board text added: "Tx"
- board text added: "v0 2017-04-23 A. Bolin"
